File: SensorHub/SensorHub_2.0/SensorHub_2.0.kicad_sch (KiCad schematic)
At the start: 56 parts, among them J1 Conn_01x02, J4 USB_C_Receptacle, P1 BM46B-12DP-0.35V_53_, P2 BM46B-12DP-0.35V_53_, U1 R7FA4E2B93CFM#AA0, U2 MYRGM080200C41RA, U3 TJA1051TK-3, U4 BMI270, U5 ASCODV-24.000MHZ-LR-T3

Commit message: Audio jumper
Parts:
- added C19: 1 uF, Capacitor_SMD:C_0603_1608Metric, symbol Device:C
- added JP1: SolderJumper_2_Open, Jumper:SolderJumper-2_P1.3mm_Open_RoundedPad1.0x1.5mm, symbol Jumper:SolderJumper_2_Open
Connections:
- net GND: now also JP1.1 (A); no longer C12.2
- net ADC/DA: now reaches U1.53 (P014)
- net ADC/DA: now also C19.1
- net ADC: no longer names the net of U1.64 (P000)
- net ADC: no longer R11.2
- new net: C12.2, JP1.2 (B)
- new net: C19.2, R11.2
Other:
- note added: "Short for ADC"
- moved on the sheet: C12, R11
Changed lines of the file:
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@@
 		)
 	)
+	(text "Short \nfor ADC\n"
+		(exclude_from_sim no)
+		(at 137.668 144.78 0)
+		(effects
+			(font
+				(size 1.27 1.27)
+			)
+		)
+	)
 	(text "Pull-Up\n(optional)"
 		(exclude_from_sim no)
@@
 	)
 	(junction
-		(at 154.94 184.15)
+		(at 132.08 130.81)
 		(diameter 0)
 		(color 0 0 0 0)
 	)
 	(junction
-		(at 208.28 48.26)
+		(at 154.94 184.15)
 		(diameter 0)
 		(color 0 0 0 0)
 	)
 	(junction
-		(at 119.38 36.83)
+		(at 208.28 48.26)
 		(diameter 0)
 		(color 0 0 0 0)
 	)
 	(junction
-		(at 132.08 134.62)
+		(at 119.38 36.83)
 		(diameter 0)
 		(color 0 0 0 0)
@@
 		)
 	)
+	(wire
+		(pts
+			(xy 132.08 129.54) (xy 132.08 130.81)
+		)
+		(stroke
+			(width 0)
+			(type default)
+		)
+	)
 	(polyline
 		(pts
@@
 		)
 	)
-	(wire
-		(pts
-			(xy 132.08 116.84) (xy 132.08 123.19)
-		)
-		(stroke
-			(width 0)
-			(type default)
-		)
-	)
 	(polyline
 		(pts
@@
 	(wire
 		(pts
+			(xy 132.08 130.81) (xy 140.97 130.81)
+		)
+		(stroke
+			(width 0)
+			(type default)
+		)
+	)
+	(wire
+		(pts
 			(xy 64.77 166.37) (xy 64.77 160.02)
 		)
@@
 	(wire
 		(pts
-			(xy 132.08 134.62) (xy 140.97 134.62)
-		)
-		(stroke
-			(width 0)
-			(type default)
-		)
-	)
-	(wire
-		(pts
 			(xy 86.36 142.24) (xy 86.36 134.62)
 		)
@@
 	(wire
 		(pts
-			(xy 132.08 130.81) (xy 132.08 134.62)
-		)
-		(stroke
-			(width 0)
-			(type default)
-		)
-	)
-	(wire
-		(pts
 			(xy 154.94 162.56) (xy 154.94 161.29)
 		)
@@
 		)
 	)
+	(label "ADC{slash}DA"
+		(at 208.28 142.24 180)
+		(effects
+			(font
+				(size 1.27 1.27)
+			)
+			(justify right bottom)
+		)
+	)
 	(label "+5V"
 		(at 86.36 25.4 180)
@@
 		)
 	)
+	(label "ADC{slash}DA"
+		(at 132.08 114.3 0)
+		(effects
+			(font
+				(size 1.27 1.27)
+			)
+			(justify left bottom)
+		)
+	)
 	(label "+5V"
 		(at 59.69 123.19 180)
@@
 		)
 	)
-	(label "ADC"
-		(at 208.28 119.38 180)
-		(effects
-			(font
-				(size 1.27 1.27)
-			)
-			(justify right bottom)
-		)
-	)
 	(label "SCL_0"
 		(at 148.59 50.8 90)
@@
 		)
 	)
-	(label "ADC"
-		(at 132.08 116.84 0)
-		(effects
-			(font
-				(size 1.27 1.27)
-			)
-			(justify left bottom)
-		)
-	)
 	(label "INT1"
 		(at 52.07 95.25 0)
@@
 	)
 	(label "Analog"
-		(at 140.97 134.62 180)
+		(at 140.97 130.81 180)
 		(effects
 			(font
@@
 	)
 	(symbol
+		(lib_id "Jumper:SolderJumper_2_Open")
+		(at 132.08 142.24 90)
+		(unit 1)
+		(exclude_from_sim no)
+		(in_bom no)
+		(on_board yes)
+		(dnp no)
+		(property "Reference" "JP1"
+			(at 134.62 140.9699 90)
+			(effects
+				(font
+					(size 1.27 1.27)
+				)
+				(justify right)
+			)
+		)
+		(property "Value" "SolderJumper_2_Open"
+			(at 134.62 148.59 90)
+			(effects
+				(font
+					(size 1.27 1.27)
+				)
+				(justify right)
+			)
+		)
+		(property "Footprint" "Jumper:SolderJumper-2_P1.3mm_Open_RoundedPad1.0x1.5mm"
+			(at 132.08 142.24 0)
+			(effects
+				(font
+					(size 1.27 1.27)
+				)
+				(hide yes)
+			)
+		)
+		(property "Datasheet" "~"
+			(at 132.08 142.24 0)
+			(effects
+				(font
+					(size 1.27 1.27)
+				)
+				(hide yes)
+			)
+		)
+		(property "Description" "Solder Jumper, 2-pole, open"
+			(at 132.08 142.24 0)
+			(effects
+				(font
+					(size 1.27 1.27)
+				)
+				(hide yes)
+			)
+		)
+		(pin "1"
+		)
+		(pin "2"
+		)
+		(instances
+			(project "SensorHub_2.0"
+				(path "/9668bc71-8924-498e-982f-628f3083c8b8"
+					(reference "JP1")
+					(unit 1)
+				)
+			)
+		)
+	)
+	(symbol
 		(lib_id "SensorHub MicroMod Carrier v1.1.0b-eagle-import:microbuilder_GND")
 		(at 90.17 191.77 0)
@@
 	(symbol
 		(lib_id "Device:C")
-		(at 132.08 138.43 0)
+		(at 132.08 134.62 0)
 		(unit 1)
 		(exclude_from_sim no)
@@
 		(fields_autoplaced yes)
 		(property "Reference" "C12"
-			(at 135.89 137.1599 0)
+			(at 135.89 133.3499 0)
 			(effects
 				(font
@@
 		)
 		(property "Value" "0.1 uF"
-			(at 135.89 139.6999 0)
+			(at 135.89 135.8899 0)
 			(effects
 				(font
@@
 		)
 		(property "Footprint" "Capacitor_SMD:C_0603_1608Metric"
-			(at 133.0452 142.24 0)
+			(at 133.0452 138.43 0)
 			(effects
 				(font
@@
 		)
 		(property "Datasheet" "~"
-			(at 132.08 138.43 0)
+			(at 132.08 134.62 0)
 			(effects
 				(font
@@
 		)
 		(property "Description" "Unpolarized capacitor"
-			(at 132.08 138.43 0)
+			(at 132.08 134.62 0)
 			(effects
 				(font
@@
 	(symbol
 		(lib_id "SensorHub MicroMod Carrier v1.1.0b-eagle-import:microbuilder_GND")
-		(at 132.08 144.78 0)
+		(at 132.08 148.59 0)
 		(unit 1)
 		(exclude_from_sim no)
@@
 		(dnp no)
 		(property "Reference" "#U$016"
-			(at 132.08 144.78 0)
+			(at 132.08 148.59 0)
 			(effects
 				(font
@@
 		)
 		(property "Value" "GND"
-			(at 130.556 147.32 0)
+			(at 130.556 151.13 0)
 			(effects
 				(font
@@
 		)
 		(property "Footprint" ""
-			(at 132.08 144.78 0)
+			(at 132.08 148.59 0)
 			(effects
 				(font
@@
 		)
 		(property "Datasheet" ""
-			(at 132.08 144.78 0)
+			(at 132.08 148.59 0)
 			(effects
 				(font
@@
 		)
 		(property "Description" ""
-			(at 132.08 144.78 0)
+			(at 132.08 148.59 0)
 			(effects
 				(font
@@
 	(symbol
 		(lib_id "Device:R")
-		(at 132.08 127 180)
+		(at 132.08 125.73 180)
 		(unit 1)
 		(exclude_from_sim no)
@@
 		(dnp no)
 		(property "Reference" "R11"
-			(at 135.89 127 90)
+			(at 135.89 125.73 90)
 			(effects
 				(font
@@
 		)
 		(property "Value" "1 K"
-			(at 134.366 126.746 90)
+			(at 134.366 125.476 90)
 			(effects
 				(font
@@
 		)
 		(property "Footprint" "Resistor_SMD:R_0201_0603Metric"
-			(at 133.858 127 90)
+			(at 133.858 125.73 90)
 			(effects
 				(font
@@
 		)
 		(property "Datasheet" "~"
-			(at 132.08 127 0)
+			(at 132.08 125.73 0)
 			(effects
 				(font
@@
 		)
 		(property "Description" "Resistor"
-			(at 132.08 127 0)
+			(at 132.08 125.73 0)
 			(effects
 				(font
@@
 					(unit 1)
 				)
+			)
+		)
+	)
+	(symbol
+		(lib_id "Device:C")
+		(at 132.08 118.11 0)
+		(unit 1)
+		(exclude_from_sim no)
+		(in_bom yes)
+		(on_board yes)
+		(dnp no)
+		(fields_autoplaced yes)
+		(property "Reference" "C19"
+			(at 135.89 116.8399 0)
+			(effects
+				(font
+					(size 1.27 1.27)
+				)
+				(justify left)
+			)
+		)
+		(property "Value" "1 uF"
+			(at 135.89 119.3799 0)
+			(effects
+				(font
+					(size 1.27 1.27)
+				)
+				(justify left)
+			)
+		)
+		(property "Footprint" "Capacitor_SMD:C_0603_1608Metric"
+			(at 133.0452 121.92 0)
+			(effects
+				(font
+					(size 1.27 1.27)
+				)
+				(hide yes)
+			)
+		)
+		(property "Datasheet" "~"
+			(at 132.08 118.11 0)
+			(effects
+				(font
+					(size 1.27 1.27)
+				)
+				(hide yes)
+			)
+		)
+		(property "Description" "Unpolarized capacitor"
+			(at 132.08 118.11 0)
+			(effects
+				(font
+					(size 1.27 1.27)
+				)
+				(hide yes)
+			)
+		)
+		(pin "1"
+		)
+		(pin "2"
+		)
+		(instances
+			(project "SensorHub_2.0"
+				(path "/9668bc71-8924-498e-982f-628f3083c8b8"
+					(reference "C19")
+					(unit 1)
+				)
