File: SensorHub/SensorHub_2.0/SensorHub_2.0.kicad_sch (KiCad schematic)
At the start: 8 parts, among them J2 658561423020, J3 658561423020

Commit message: PCB_1.0
Other:
- sheet RA4E2_microcontroller ports: added Sleep; removed none
Changed lines of the file:
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@@
-		)
-	)
-	(label "+5V"
-		(at 67.31 124.46 0)
-		(effects
-			(font
-				(size 1.27 1.27)
-			)
-			(justify left bottom)
 		)
 	)
@@
 			)
 			(justify left bottom)
-		)
-	)
-	(label "+5V"
-		(at 34.29 124.46 180)
-		(effects
-			(font
-				(size 1.27 1.27)
-			)
-			(justify right bottom)
 		)
 	)
@@
 				(path "/9668bc71-8924-498e-982f-628f3083c8b8"
 					(reference "JP1")
+					(unit 1)
+				)
+			)
+		)
+	)
+	(symbol
+		(lib_id "power:+5V")
+		(at 67.31 124.46 270)
+		(unit 1)
+		(exclude_from_sim no)
+		(in_bom yes)
+		(on_board yes)
+		(dnp no)
+		(fields_autoplaced yes)
+		(property "Reference" "#PWR047"
+			(at 63.5 124.46 0)
+			(effects
+				(font
+					(size 1.27 1.27)
+				)
+				(hide yes)
+			)
+		)
+		(property "Value" "+5V"
+			(at 71.12 124.4599 90)
+			(effects
+				(font
+					(size 1.27 1.27)
+				)
+				(justify left)
+			)
+		)
+		(property "Footprint" ""
+			(at 67.31 124.46 0)
+			(effects
+				(font
+					(size 1.27 1.27)
+				)
+				(hide yes)
+			)
+		)
+		(property "Datasheet" ""
+			(at 67.31 124.46 0)
+			(effects
+				(font
+					(size 1.27 1.27)
+				)
+				(hide yes)
+			)
+		)
+		(property "Description" "Power symbol creates a global label with name \"+5V\""
+			(at 67.31 124.46 0)
+			(effects
+				(font
+					(size 1.27 1.27)
+				)
+				(hide yes)
+			)
+		)
+		(pin "1"
+		)
+		(instances
+			(project "SensorHub_2.0"
+				(path "/9668bc71-8924-498e-982f-628f3083c8b8"
+					(reference "#PWR047")
 					(unit 1)
 				)
@@
 	)
 	(symbol
+		(lib_id "power:GND")
+		(at 90.17 146.05 0)
+		(unit 1)
+		(exclude_from_sim no)
+		(in_bom yes)
+		(on_board yes)
+		(dnp no)
+		(fields_autoplaced yes)
+		(property "Reference" "#PWR048"
+			(at 90.17 152.4 0)
+			(effects
+				(font
+					(size 1.27 1.27)
+				)
+				(hide yes)
+			)
+		)
+		(property "Value" "GND"
+			(at 90.17 151.13 0)
+			(effects
+				(font
+					(size 1.27 1.27)
+				)
+			)
+		)
+		(property "Footprint" ""
+			(at 90.17 146.05 0)
+			(effects
+				(font
+					(size 1.27 1.27)
+				)
+				(hide yes)
+			)
+		)
+		(property "Datasheet" ""
+			(at 90.17 146.05 0)
+			(effects
+				(font
+					(size 1.27 1.27)
+				)
+				(hide yes)
+			)
+		)
+		(property "Description" "Power symbol creates a global label with name \"GND\" , ground"
+			(at 90.17 146.05 0)
+			(effects
+				(font
+					(size 1.27 1.27)
+				)
+				(hide yes)
+			)
+		)
+		(pin "1"
+		)
+		(instances
+			(project "SensorHub_2.0"
+				(path "/9668bc71-8924-498e-982f-628f3083c8b8"
+					(reference "#PWR048")
+					(unit 1)
+				)
+			)
+		)
+	)
+	(symbol
 		(lib_id "Device:C")
 		(at 90.17 134.62 0)
@@
 	)
 	(symbol
-		(lib_id "SensorHub MicroMod Carrier v1.1.0b-eagle-import:microbuilder_GND")
-		(at 90.17 148.59 0)
+		(lib_id "power:+5V")
+		(at 34.29 124.46 90)
 		(unit 1)
 		(exclude_from_sim no)
@@
 		(on_board yes)
 		(dnp no)
-		(property "Reference" "#U$016"
-			(at 90.17 148.59 0)
-			(effects
-				(font
-					(size 1.27 1.27)
-				)
-				(hide yes)
-			)
-		)
-		(property "Value" "GND"
-			(at 88.646 151.13 0)
-			(effects
-				(font
-					(size 1.27 1.0795)
-				)
-				(justify left bottom)
+		(fields_autoplaced yes)
+		(property "Reference" "#PWR046"
+			(at 38.1 124.46 0)
+			(effects
+				(font
+					(size 1.27 1.27)
+				)
+				(hide yes)
+			)
+		)
+		(property "Value" "+5V"
+			(at 30.48 124.4599 90)
+			(effects
+				(font
+					(size 1.27 1.27)
+				)
+				(justify left)
 			)
 		)
 		(property "Footprint" ""
-			(at 90.17 148.59 0)
+			(at 34.29 124.46 0)
 			(effects
 				(font
@@
 		)
 		(property "Datasheet" ""
-			(at 90.17 148.59 0)
-			(effects
-				(font
-					(size 1.27 1.27)
-				)
-				(hide yes)
-			)
-		)
-		(property "Description" ""
-			(at 90.17 148.59 0)
+			(at 34.29 124.46 0)
+			(effects
+				(font
+					(size 1.27 1.27)
+				)
+				(hide yes)
+			)
+		)
+		(property "Description" "Power symbol creates a global label with name \"+5V\""
+			(at 34.29 124.46 0)
 			(effects
 				(font
@@
 			(project "SensorHub_2.0"
 				(path "/9668bc71-8924-498e-982f-628f3083c8b8"
-					(reference "#U$016")
+					(reference "#PWR046")
 					(unit 1)
 				)
@@
 			(effects
 				(font
+					(size 1.27 1.27)
+				)
+				(justify left)
+			)
+		)
+		(pin "Sleep" input
+			(at 208.28 104.14 180)
+			(effects
+				(font

Commit message: Fix 17.04
Other:
- sheet MYRGM080200C41RA +5\+3.3 ports: added none; removed Sleep
Changed lines of the file:
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@@
 	(wire
 		(pts
-			(xy 35.56 35.56) (xy 41.91 35.56)
+			(xy 57.15 137.16) (xy 44.45 137.16)
 		)
 		(stroke
@@
 	(wire
 		(pts
-			(xy 57.15 137.16) (xy 44.45 137.16)
+			(xy 200.66 87.63) (xy 208.28 87.63)
 		)
 		(stroke
@@
 	(wire
 		(pts
-			(xy 200.66 87.63) (xy 208.28 87.63)
+			(xy 57.15 121.92) (xy 44.45 121.92)
 		)
 		(stroke
@@
 		)
 	)
-	(wire
+	(polyline
 		(pts
-			(xy 57.15 121.92) (xy 44.45 121.92)
+			(xy 281.94 15.24) (xy 281.94 163.83)
 		)
 		(stroke
@@
 		)
 	)
-	(polyline
+	(wire
 		(pts
-			(xy 281.94 15.24) (xy 281.94 163.83)
+			(xy 203.2 38.1) (xy 208.28 38.1)
 		)
 		(stroke
@@
 	(wire
 		(pts
-			(xy 203.2 38.1) (xy 208.28 38.1)
+			(xy 203.2 80.01) (xy 208.28 80.01)
 		)
 		(stroke
@@
 	(wire
 		(pts
-			(xy 203.2 80.01) (xy 208.28 80.01)
+			(xy 57.15 139.7) (xy 44.45 139.7)
 		)
 		(stroke
@@
 		)
 	)
-	(wire
+	(polyline
 		(pts
-			(xy 57.15 139.7) (xy 44.45 139.7)
+			(xy 175.26 15.24) (xy 281.94 15.24)
 		)
 		(stroke
@@
 		)
 	)
-	(polyline
+	(wire
 		(pts
-			(xy 175.26 15.24) (xy 281.94 15.24)
+			(xy 57.15 134.62) (xy 44.45 134.62)
 		)
 		(stroke
@@
 		)
 	)
+	(polyline
+		(pts
+			(xy 139.7 152.4) (xy 175.26 152.4)
+		)
+		(stroke
+			(width 0)
+			(type solid)
+		)
+	)
 	(wire
 		(pts
-			(xy 57.15 134.62) (xy 44.45 134.62)
+			(xy 200.66 85.09) (xy 208.28 85.09)
 		)
 		(stroke
@@
 	(polyline
 		(pts
-			(xy 139.7 152.4) (xy 175.26 152.4)
+			(xy 102.87 152.4) (xy 102.87 109.22)
 		)
 		(stroke
@@
 	(wire
 		(pts
-			(xy 200.66 85.09) (xy 208.28 85.09)
+			(xy 57.15 127) (xy 44.45 127)
 		)
 		(stroke
@@
 		)
 	)
+	(wire
+		(pts
+			(xy 57.15 132.08) (xy 44.45 132.08)
+		)
+		(stroke
+			(width 0)
+			(type default)
+		)
+	)
+	(wire
+		(pts
+			(xy 90.17 129.54) (xy 90.17 130.81)
+		)
+		(stroke
+			(width 0)
+			(type default)
+		)
+	)
 	(polyline
 		(pts
-			(xy 102.87 152.4) (xy 102.87 109.22)
+			(xy 34.29 152.4) (xy 102.87 152.4)
 		)
 		(stroke
@@
 	(wire
 		(pts
-			(xy 57.15 127) (xy 44.45 127)
+			(xy 204.47 96.52) (xy 208.28 96.52)
 		)
 		(stroke
@@
 		)
 	)
-	(wire
-		(pts
-			(xy 57.15 132.08) (xy 44.45 132.08)
-		)
-		(stroke
-			(width 0)
-			(type default)
-		)
-	)
-	(wire
-		(pts
-			(xy 90.17 129.54) (xy 90.17 130.81)
-		)
-		(stroke
-			(width 0)
-			(type default)
-		)
-	)
-	(polyline
-		(pts
-			(xy 34.29 152.4) (xy 102.87 152.4)
-		)
-		(stroke
-			(width 0)
-			(type solid)
-		)
-	)
-	(wire
-		(pts
-			(xy 204.47 96.52) (xy 208.28 96.52)
-		)
-		(stroke
-			(width 0)
-			(type default)
-		)
-	)
 	(label "SCL_0"
 		(at 46.99 55.88 180)
@@
 			)
 			(justify left bottom)
-		)
-	)
-	(label "Sleep"
-		(at 41.91 35.56 180)
-		(effects
-			(font
-				(size 1.27 1.27)
-			)
-			(justify right bottom)
 		)
 	)
@@
 			)
 		)
-		(pin "Sleep" bidirectional
-			(at 35.56 35.56 0)
-			(effects
-				(font
-					(size 1.27 1.27)
-				)
-				(justify right)
-			)
-		)
