File: SensorHub/SensorHub_2.0/SensorHub_2.0.kicad_sch (KiCad schematic)
At the start: 8 parts, among them J2 658561423020, J3 658561423020

Commit message: Fix2 17.04
Connections:
- no-connect marks 0 -> 1
Changed lines of the file:
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@@
 		(color 0 0 0 0)
+	)
+	(no_connect
+		(at 208.28 104.14)
 	)
 	(polyline

Commit message: PCB fix
Connections:
- no-connect marks 1 -> 3
Other:
- removed sheet USB_C_2.0+SBUS
- added sheet USB_C_3.0 (USB_C_3.0.kicad_sch)

Commit message: Vesrion 2
Parts:
- added C22, C23, C5: 0.1 uF, Capacitor_SMD:C_0603_1608Metric, symbol Device:C
- added U5, U8: USBLC6-4SC6, Package_TO_SOT_SMD:SOT-23-6, symbol Power_Protection:USBLC6-4SC6
- TP2, TP7: footprint TestPoint:TestPoint_THTPad_D1.0mm_Drill0.5mm -> TestPoint:TestPoint_Pad_1.0x1.0mm
Connections:
- net +3.3V: now also C22.1, C5.1, U5.5 (VBUS), U8.5 (VBUS)
- net +5V: now also C23.1
- net Analog: now also U5.1 (I/O1)
- net CS: now also U8.4 (I/O3)
- net GND: now also C22.2, C23.2, C5.2, U5.2 (GND), U8.2 (GND)
- net INT2: now also U5.3 (I/O2)
- net MISO: now also U8.1 (I/O1)
- net MOSI: now also U8.3 (I/O2)
- net SCK: now also U8.6 (I/O4)
- net SCL_0: now also U5.4 (I/O3)
- net SDA_0: now also U5.6 (I/O4)
- no-connect marks 3 -> 1
Other:
- removed sheet USB_C_3.0
- added sheet USB_C_2.0+SBUS (USB_C_2.0+SBUS.kicad_sch)
- sheet CAN_transeiver ports: added STB; removed none
- note removed: "20.03.2026"
- note removed: "Design by Artur Erik"
- title: (none) -> SensorHub_2.0_ManikinSystem26
- moved on the sheet: C12, C19, JP1, R11, TP2, TP7

Commit message: MPN + CC fix
Parts:
- J2, J3: MPN (none) -> 658561423020
- U5, U8: MPN (none) -> USBLC6-4SC6Y
Changed lines of the file:
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@@
+			)
+		)
+		(property "MPN" "658561423020"
+			(at 62.23 133.35 90)
+			(effects
+				(font
+					(size 1.27 1.27)
+				)
+				(hide yes)
 			)
 		)
@@
 			)
 		)
+		(property "MPN" "658561423020"
+			(at 39.37 133.35 90)
+			(effects
+				(font
+					(size 1.27 1.27)
+				)
+				(hide yes)
+			)
+		)
 		(pin "14"
 		)
@@
 			)
 		)
+		(property "MPN" "USBLC6-4SC6Y "
+			(at 154.94 151.13 0)
+			(effects
+				(font
+					(size 1.27 1.27)
+				)
+				(hide yes)
+			)
+		)
 		(pin "6"
 		)
@@
 			(at 154.94 123.19 0)
 			(effects
+				(font
+					(size 1.27 1.27)
+				)
+				(hide yes)
+			)
+		)
+		(property "MPN" "USBLC6-4SC6Y "
+			(at 154.94 123.19 0)
+			(effects

Commit message: pcb fix
Parts:
- R11: footprint Resistor_SMD:R_0201_0603Metric -> Resistor_SMD:R_0402_1005Metric
Changed lines of the file:
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@@
 			)
 		)
-		(property "Footprint" "Resistor_SMD:R_0201_0603Metric"
+		(property "Footprint" "Resistor_SMD:R_0402_1005Metric"
 			(at 123.698 125.73 90)
 			(effects

Commit message: v 2.3
Parts:
- R11: footprint Resistor_SMD:R_0402_1005Metric -> Resistor_SMD:R_0603_1608Metric
Connections:
- net Analog: now also U5.4 (I/O3); no longer U5.1 (I/O1)
- net CS: now also U8.6 (I/O4); no longer U8.4 (I/O3)
- net MISO: now also U8.3 (I/O2); no longer U8.1 (I/O1)
- net MOSI: now also U8.1 (I/O1); no longer U8.3 (I/O2)
- net SCK: now also U8.4 (I/O3); no longer U8.6 (I/O4)
- net SCL_0: now also U5.6 (I/O4); no longer U5.4 (I/O3)
- net SDA_0: now also U5.1 (I/O1); no longer U5.6 (I/O4)
Other:
- title: SensorHub_2.0_ManikinSystem26 -> SensorHub_2.3_ManikinSystem26
Changed lines of the file:
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@@
 	(paper "A4")
 	(title_block
-		(title "SensorHub_2.0_ManikinSystem26")
+		(title "SensorHub_2.3_ManikinSystem26")
 		(date "28.04.2026")
 		(comment 4 "Design by Artur Erik")
@@
 	)
 	(label "SCK"
-		(at 147.32 128.27 180)
+		(at 147.32 125.73 180)
 		(effects
 			(font
@@
 	)
 	(label "SCL_0"
-		(at 147.32 153.67 180)
+		(at 147.32 156.21 180)
 		(effects
 			(font
@@
 	)
 	(label "SDA_0"
-		(at 147.32 156.21 180)
+		(at 147.32 148.59 180)
 		(effects
 			(font
@@
 	)
 	(label "MISO"
-		(at 147.32 120.65 180)
+		(at 147.32 123.19 180)
 		(effects
 			(font
@@
 	)
 	(label "CS"
-		(at 147.32 125.73 180)
+		(at 147.32 128.27 180)
 		(effects
 			(font
@@
 	)
 	(label "MOSI"
-		(at 147.32 123.19 180)
+		(at 147.32 120.65 180)
 		(effects
 			(font
@@
 	)
 	(label "Analog"
-		(at 147.32 148.59 180)
+		(at 147.32 153.67 180)
 		(effects
 			(font
@@
 			)
 		)
-		(property "Footprint" "Resistor_SMD:R_0402_1005Metric"
+		(property "Footprint" "Resistor_SMD:R_0603_1608Metric"
 			(at 123.698 125.73 90)
 			(effects
