File: SensorHub/SensorHub_2.0/RA4E2_microcontroller.kicad_sch (KiCad schematic)
At the start: 30 parts, among them J1 Conn_01x02, U1 R7FA4E2B93CFM#AA0, U5 ASCODV-24.000MHZ-LR-T3

Commit message: TCAN334
Parts:
- removed C15: 0.1 uF, Capacitor_SMD:C_0603_1608Metric, symbol Device:C
- removed J1: Conn_01x02, Connector_PinSocket_1.00mm:PinSocket_1x02_P1.00mm_Vertical, symbol Connector_Generic:Conn_01x02
- removed TP1, TP2, TP7: TestPoint, TestPoint:TestPoint_THTPad_D1.0mm_Drill0.5mm, symbol Connector:TestPoint
- added J5: Conn_02x05_Top_Bottom, Connector_PinHeader_1.00mm:PinHeader_2x05_P1.00mm_Vertical, symbol Connector_Generic:Conn_02x05_Top_Bottom
Connections:
- net +3.3V: now also J5.1 (Pin_1)
- net GND: now also J5.10 (Pin_10), J5.2 (Pin_2), J5.4 (Pin_4), J5.6 (Pin_6), J5.8 (Pin_8)
- net RES: now also J5.5 (Pin_5)
- net SWCLK: now also J5.9 (Pin_9)
- net SWDIO: now also J5.7 (Pin_7)
- net TXD: no longer U1.12 (P411)
- net VCL: now also J5.3 (Pin_3)
Other:
- moved on the sheet: C10, C11, C13, C14, C5, C7, D1, D2, R15, R3, R4, R5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

Commit message: 32k oscillator
Parts:
- removed D1, D2: LED, LED_SMD:LED_0402_1005Metric, symbol Device:LED
- removed R3, R8: 1.33 K, Resistor_SMD:R_0201_0603Metric, symbol Device:R
- removed U5: ASCODV-24.000MHZ-LR-T3, Library:ASCODV-24.000MHZ-LR-T3, symbol Library:ASCODV-24.000MHZ-LR-T3
- added C15, C9: 0.1 uF, Capacitor_SMD:C_0603_1608Metric, symbol Device:C
- added D4, D5: 1312020030000, 1312020030000:1312020030000, symbol 1312020030000:1312020030000
- added Y1: ASH7KW-32.768KHZ-L-T, ASH7KW-32.768KHZ-L-T:XTAL_ASH7KW-32.768KHZ-L-T, symbol ASH7KW-32.768KHZ-L-T:ASH7KW-32.768KHZ-L-T
Connections:
- net +3.3V: now also C16.1, Y1.3 (OE), Y1.4 (VDD)
- net EXTAL: now also Y1.1 (OUTPUT)
- net GND: now also C15.2, C9.2, D4.4, D5.4, Y1.2 (GND)
- net LED1 renamed LED
- net LED: now also D5.3
- net LED2: no longer names the net of U1.22 (P206)
- new net: C9.1, D4.2
- new net: D4.3, D5.1
- new net: C15.1, D5.2
- no-connect marks 0 -> 1
Other:
- moved on the sheet: C16, J5, TP3, TP4, TP5, TP6, TP8

Commit message: FTSH
Parts:
- removed J5: Conn_02x05_Top_Bottom, Connector_PinHeader_1.00mm:PinHeader_2x05_P1.00mm_Vertical, symbol Connector_Generic:Conn_02x05_Top_Bottom
- added J5: FTSH-105-01-L-DV-K-A, FTSH-105-01-L-DV-K-A:SAMTEC_FTSH-105-01-L-DV-K-A, symbol FTSH-105-01-L-DV-K-A:FTSH-105-01-L-DV-K-A
Connections:
- net +3.3V: now also J5.01
- net GND: now also J5.03, J5.05, J5.09
- net RES: now also J5.10
- net SWCLK: now also J5.04
- net SWDIO: now also J5.02
- no-connect marks 1 -> 4
Other:
- moved on the sheet: TP3, TP4, TP5, TP6, TP8

Commit message: New_USB_2.0
Parts:
- removed S1: Reset, Library:Button_Mini_2.5x1.7mm, symbol SensorHub MicroMod Carrier v1.1.0b-eagle-import:MOMENTARY-SWITCH-SPST-SMD-5.2-T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
- removed S2: Boot, Library:Button_Mini_2.5x1.7mm, symbol SensorHub MicroMod Carrier v1.1.0b-eagle-import:MOMENTARY-SWITCH-SPST-SMD-5.2-T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
- added SW1, SW2: SW_Push, Library:B3U-1000P(M)-B, symbol Library:SW_Push
- added TP1: TestPoint, TestPoint:TestPoint_THTPad_D1.0mm_Drill0.5mm, symbol Connector:TestPoint
Connections:
- net Boot: now also SW2.2
- net GND: now also SW1.1
- net RES: now also SW1.2, TP1.1
- net at R5.1: now also SW2.1
- net GP3: now reaches U1.12 (P411)
- net GP2: now reaches U1.13 (P410)
Other:
- moved on the sheet: C7, R4, R6

Commit message: PCB 1st upd
Parts:
- added C17, C18: 0.1 uF, Capacitor_SMD:C_0603_1608Metric, symbol Device:C
Connections:
- net +3.3V: now also C17.1, C18.1
- net GND: now also C17.2, C18.2
- net SWCLK: now also J5.02; no longer J5.04
- net SWDIO: now also J5.04; no longer J5.02
- no-connect marks 4 -> 37

Commit message: PCB upd 2
Connections:
- net INT1: now also U1.1 (P400); no longer U1.44 (P104)
- net INT2: now also U1.44 (P104); no longer U1.1 (P400)
Changed lines of the file:
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@@
-		)
-	)
-	(hierarchical_label "INT1"
-		(shape input)
-		(at 246.38 54.61 0)
-		(effects
-			(font
-				(size 1.27 1.27)
-			)
-			(justify left)
 		)
 	)
@@
 		)
 	)
-	(hierarchical_label "INT2"
+	(hierarchical_label "INT1"
 		(shape input)
 		(at 246.38 100.33 0)
@@
 		)
 	)
+	(hierarchical_label "INT2"
+		(shape input)
+		(at 246.38 54.61 0)
+		(effects
+			(font
+				(size 1.27 1.27)
+			)
+			(justify left)
+		)
+	)

Commit message: PCB_1.0
Parts:
- removed C5: 0.1 uF, Capacitor_SMD:C_0603_1608Metric, symbol Device:C
- added TP10: TestPoint, TestPoint:TestPoint_THTPad_D1.0mm_Drill0.5mm, symbol Connector:TestPoint
Connections:
- net Boot: now also TP1.1; no longer TP5.1
- net GND: now also TP10.1
- net GP2: now also U1.30 (P302); no longer U1.13 (P410)
- net GP3: now also U1.29 (P303); no longer U1.12 (P411)
- net RES: now also TP5.1; no longer TP1.1
- net SCL_0: now also TP4.1; no longer TP3.1
- net SDA_0: now also TP3.1; no longer TP4.1
- net Sleep: now reaches U1.41 (P107)
- no-connect marks 37 -> 36
Other:
- moved on the sheet: C13, C14, C17, C18
