File: SensorHub/SensorHub_2.0/SensorHub_2.0.kicad_pcb (KiCad board)
At the start: 4 copper layers, 30 x 28 mm, 67 parts, among them J2 658561423020, J3 658561423020, J5 FTSH-105-01-L-DV-K-A, J6 USB_C_Receptacle_USB2.0_16P, J8 USB_C_Receptacle_USB2.0_16P, U1 R7FA4E2B93CFM#AA0, U10 LMV339, U2 MYRGM080200C41RA, U3 TCAN334, U4 USBLC6-4SC6, U5 TMUX154EDGS, U6 LSM6DSM, U7 USBLC6-4SC6, Y1 ASH7KW-32.768KHZ-L-T

Commit message: Fix 17.04
Parts:
- renumbered RES to SW1, Boot to SW2, |Boot to TP1, GND to TP10, GP3 to TP2, SDA to TP3, SCL to TP4, RES to TP5, EXTAL to TP6, GP2 to TP7, TXD to TP8
Connections:
- J2 pad 2: /+3.3V -> +3.3V
- J3 pad 12: /+3.3V -> +3.3V
Routing:
- net +3.3V: track 40.2 -> 42.4 mm, vias 17 -> 18
- net GND: track 106.1 -> 104.1 mm, vias 42 -> 41
- net /+3.3V: track 1.93 -> 0.00 mm, vias 1 -> 0
Changed lines of the file:
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@@
 	(net 92 "Net-(U2-CE)")
 	(net 93 "/RA4E2_microcontroller/Sleep")
-	(net 94 "/+3.3V")
 	(footprint "FTSH-105-01-L-DV-K-A:SAMTEC_FTSH-105-01-L-DV-K-A"
 		(layer "F.Cu")
@@
 			(size 0.25 1.1)
 			(layers "F.Cu" "F.Mask" "F.Paste")
-			(net 94 "/+3.3V")
+			(net 39 "+3.3V")
 			(pinfunction "2")
 			(pintype "passive")
@@
 		(descr "THT pad as test Point, diameter 1.0mm, hole diameter 0.5mm")
 		(tags "test point THT pad")
-		(property "Reference" "GP2"
+		(property "Reference" "TP7"
 			(at 0 -1.448 0)
 			(layer "F.SilkS")
@@
 		(descr "THT pad as test Point, diameter 1.0mm, hole diameter 0.5mm")
 		(tags "test point THT pad")
-		(property "Reference" "SDA"
+		(property "Reference" "TP3"
 			(at -1.9 0 0)
 			(layer "F.SilkS")
@@
 		(descr "THT pad as test Point, diameter 1.0mm, hole diameter 0.5mm")
 		(tags "test point THT pad")
-		(property "Reference" "EXTAL"
+		(property "Reference" "TP6"
 			(at 2.2 -0.8 0)
 			(layer "F.SilkS")
@@
 		(descr "THT pad as test Point, diameter 1.0mm, hole diameter 0.5mm")
 		(tags "test point THT pad")
-		(property "Reference" "RES"
+		(property "Reference" "TP5"
 			(at -0.3 1.5 0)
 			(layer "F.SilkS")
@@
 		(layer "F.Cu")
 		(at 144.799999 73.19)
-		(property "Reference" "Boot"
+		(property "Reference" "SW2"
 			(at -2.499999 -1.09 0)
 			(unlocked yes)
@@
 		(descr "THT pad as test Point, diameter 1.0mm, hole diameter 0.5mm")
 		(tags "test point THT pad")
-		(property "Reference" "GND"
+		(property "Reference" "TP10"
 			(at 0 -1.448 0)
 			(layer "F.SilkS")
@@
 		(descr "THT pad as test Point, diameter 1.0mm, hole diameter 0.5mm")
 		(tags "test point THT pad")
-		(property "Reference" "GP3"
+		(property "Reference" "TP2"
 			(at 0 -1.448 0)
 			(layer "F.SilkS")
@@
 		(layer "F.Cu")
 		(at 144.799999 76.09)
-		(property "Reference" "RES"
+		(property "Reference" "SW1"
 			(at -2.199999 -1.19 0)
 			(unlocked yes)
@@
 		(descr "THT pad as test Point, diameter 1.0mm, hole diameter 0.5mm")
 		(tags "test point THT pad")
-		(property "Reference" "TXD"
+		(property "Reference" "TP8"
 			(at -1.9 0 0)
 			(layer "F.SilkS")
@@
 		(descr "THT pad as test Point, diameter 1.0mm, hole diameter 0.5mm")
 		(tags "test point THT pad")
-		(property "Reference" "SCL"
+		(property "Reference" "TP4"
 			(at -1.9 0 0)
 			(layer "F.SilkS")
@@
 		(descr "THT pad as test Point, diameter 1.0mm, hole diameter 0.5mm")
 		(tags "test point THT pad")
-		(property "Reference" "|Boot"
+		(property "Reference" "TP1"
 			(at 0.1 1.5 0)
 			(layer "F.SilkS")
@@
 	(footprint "Connector_SMD_Wurth:J_Wurth_WR-BTB_658561423020"
 		(layer "B.Cu")
-		(at 159.498999 94.39 180)
+		(at 159.498999 94.35 180)
 		(descr "BTB 0,4mm Vertical Plug, body 7.6x5x1.4mm, https://www.we-online.com/en/components/products/datasheet/658561423020?ki")
 		(tags "MaleHeader Vertical")
@@
 			(size 0.25 1.1)
 			(layers "B.Cu" "B.Mask" "B.Paste")
-			(net 94 "/+3.3V")
+			(net 39 "+3.3V")
 			(pinfunction "12")
 			(pintype "passive")
@@
 	)
 	(segment
-		(start 161.770076 98.079178)
-		(end 161.770076 97.132636)
-		(width 0.2)
-		(layer "F.Cu")
-		(net 30)
-	)
-	(segment
 		(start 160.755935 91.621072)
 		(end 160.755935 90.665144)
@@
 	)
 	(via
-		(at 161.754127 98.14)
-		(size 0.3)
-		(drill 0.15)
-		(layers "F.Cu" "B.Cu")
-		(net 30)
-	)
-	(via
 		(at 159.748999 90.64)
 		(size 0.3)
@@
 	)
 	(segment
-		(start 161.754127 98.14)
-		(end 161.754127 97.145128)
-		(width 0.2)
-		(layer "B.Cu")
-		(net 30)
-	)
-	(segment
 		(start 161.988999 92.15)
 		(end 162.2 92.15)
@@
 	)
 	(segment
+		(start 161.270076 98.079178)
+		(end 161.270076 97.155224)
+		(width 0.2)
+		(layer "F.Cu")
+		(net 39)
+	)
+	(segment
 		(start 141.4 92)
 		(end 141.51 91.89)
@@
 	)
 	(segment
+		(start 161.248999 97.279092)
+		(end 161.255249 97.272842)
+		(width 0.2)
+		(layer "F.Cu")
+		(net 39)
+	)
+	(segment
 		(start 161.849999 72.6775)
 		(end 160.5 72.6775)
@@
 	)
 	(via
+		(at 161.254127 98.14)
+		(size 0.3)
+		(drill 0.15)
+		(layers "F.Cu" "B.Cu")
+		(net 39)
+	)
+	(via
 		(at 148.5 94.8)
 		(size 0.6)
@@
 	)
 	(segment
+		(start 161.254127 98.14)
+		(end 161.254127 97.145128)
+		(width 0.2)
+		(layer "B.Cu")
+		(net 39)
+	)
+	(segment
 		(start 156.024999 76.09)
 		(end 156.024999 76.965)
@@
 	)
 	(segment
+		(start 161.254127 97.145128)
+		(end 161.248999 97.14)
+		(width 0.2)
+		(layer "B.Cu")
+		(net 39)
+	)
+	(segment
 		(start 152.574999 79.665)
 		(end 152.599999 79.69)
@@
 	)
 	(segment
+		(start 161.46 98.14)
+		(end 161.5 98.1)
+		(width 0.2)
+		(layer "In2.Cu")
+		(net 39)
+	)
+	(segment
+		(start 161.254127 98.14)
+		(end 161.46 98.14)
+		(width 0.2)
+		(layer "In2.Cu")
+		(net 39)
+	)
+	(segment
 		(start 155.749999 80.505)
 		(end 155.429999 80.185)
@@
 		(net 92)
 	)
-	(segment
-		(start 161.270076 98.079178)
-		(end 161.270076 97.155224)
-		(width 0.2)
-		(layer "F.Cu")
-		(net 94)
-	)
-	(segment
-		(start 161.248999 97.279092)
-		(end 161.255249 97.272842)
-		(width 0.2)
-		(layer "F.Cu")
-		(net 94)
-	)
-	(via
-		(at 161.254127 98.14)
-		(size 0.3)
-		(drill 0.15)
-		(layers "F.Cu" "B.Cu")
-		(net 94)
-	)
-	(segment
-		(start 161.254127 98.14)
-		(end 161.254127 97.145128)
-		(width 0.2)
-		(layer "B.Cu")
-		(net 94)
-	)
-	(segment
-		(start 161.254127 97.145128)
-		(end 161.248999 97.14)
-		(width 0.2)
-		(layer "B.Cu")
-		(net 94)
-	)
 	(zone

Commit message: Fix2 17.04
Routing:
- net /V_Bus: track 42.7 -> 50.3 mm, vias 1 -> 2
- net GND: track 104.1 -> 106.6 mm, vias 41 -> 42
Changed lines of the file:
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@@
 	)
 	(segment
-		(start 155.073199 80.85416)
-		(end 155.073199 80.825)
-		(width 0.2)
-		(layer "B.Cu")
-		(net 29)
-	)
-	(segment
 		(start 150.29 75.59)
 		(end 150.3 75.6)
@@
 	)
 	(segment
+		(start 157.599999 77.19)
+		(end 157.349999 76.94)
+		(width 0.3)
+		(layer "F.Cu")
+		(net 30)
+	)
+	(segment
 		(start 166.499999 78.49)
 		(end 166.359999 78.35)
@@
 	)
 	(segment
+		(start 157.349999 76.94)
+		(end 157.349999 76.065)
+		(width 0.3)
+		(layer "F.Cu")
+		(net 30)
+	)
+	(segment
 		(start 143.296999 93.085)
 		(end 143.554999 93.085)
@@
 	)
 	(via
+		(at 157.3 81.8)
+		(size 0.6)
+		(drill 0.3)
+		(layers "F.Cu" "B.Cu")
+		(net 30)
+	)
+	(via
 		(at 166.499999 79.39)
 		(size 0.6)
@@
 	)
 	(segment
+		(start 157.299999 80.505)
+		(end 157.3 81.8)
+		(width 0.4)
+		(layer "B.Cu")
+		(net 30)
+	)
+	(segment
 		(start 159.748999 92.39)
 		(end 159.7 92.438999)
@@
 	(segment
 		(start 134.582547 85.830597)
-		(end 134.582547 83.973903)
+		(end 134.582547 84.069003)
 		(width 0.3)
 		(layer "F.Cu")
@@
 	)
 	(segment
+		(start 134.582547 84.069003)
+		(end 134.582547 83.973903)
+		(width 0.3)
+		(layer "F.Cu")
+		(net 53)
+	)
+	(segment
 		(start 143.965 81.4)
 		(end 143.965 81.955)
@@
 		(net 53)
 	)
+	(via
+		(at 134.582547 84.9)
+		(size 0.3)
+		(drill 0.15)
+		(layers "F.Cu" "B.Cu")
+		(net 53)
+	)
+	(segment
+		(start 134.582547 85.84494)
+		(end 135.816607 87.079)
+		(width 0.3)
+		(layer "B.Cu")
+		(net 53)
+	)
+	(segment
+		(start 135.850087 82.701)
+		(end 134.582547 83.96854)
+		(width 0.3)
+		(layer "B.Cu")
+		(net 53)
+	)
+	(segment
+		(start 136.84355 82.49)
+		(end 136.64455 82.689)
+		(width 0.3)
+		(layer "B.Cu")
+		(net 53)
+	)
+	(segment
+		(start 135.816607 87.079)
+		(end 136.079 87.079)
+		(width 0.3)
+		(layer "B.Cu")
+		(net 53)
+	)
+	(segment
+		(start 134.582547 83.96854)
+		(end 134.582547 84.9)
+		(width 0.3)
+		(layer "B.Cu")
+		(net 53)
+	)
+	(segment
+		(start 134.582547 84.9)
+		(end 134.582547 85.84494)
+		(width 0.3)
+		(layer "B.Cu")
+		(net 53)
+	)
+	(segment
+		(start 136.29 87.29)
+		(end 136.84355 87.29)
+		(width 0.3)
+		(layer "B.Cu")
+		(net 53)
+	)
+	(segment
+		(start 136.64455 82.689)
+		(end 136.085914 82.689)
+		(width 0.3)
+		(layer "B.Cu")
+		(net 53)
+	)
+	(segment
+		(start 136.073914 82.701)
+		(end 135.850087 82.701)
+		(width 0.3)
+		(layer "B.Cu")
+		(net 53)
+	)
+	(segment
+		(start 136.079 87.079)
+		(end 136.29 87.29)
+		(width 0.3)
+		(layer "B.Cu")
+		(net 53)
+	)
 	(segment
 		(start 148.244999 81.99)
@@
 		(width 0.3)
 		(layer "B.Cu")
+		(net 53)
+	)
+	(segment
+		(start 136.085914 82.689)
+		(end 136.073914 82.701)
+		(width 0.3)
+		(layer "B.Cu")

Commit message: JLCPCB limits
Parts:
- moved C2 0.09 mm to (142.3, 89.7)
Routing:
- net GND: track 106.6 -> 108.0 mm
- net /RA4E2_microcontroller/EXTAL: track 10.4 -> 9.35 mm
- net /Can_L: vias 2 -> 1
