File: SensorHub/SensorHub_2.0/USB_C_2.0+SBUS.kicad_sch (KiCad schematic)
At the start: 10 parts, among them J6 USB_C_Receptacle_USB2.0_16P, J8 USB_C_Receptacle_USB2.0_16P, U10 LMV339, U4 USBLC6-4SC6, U5 TMUX154EDGS, U7 USBLC6-4SC6

Commit message: New_USB_2.0
Connections:
- net Can_H renamed Out_1
- net Can_L renamed Out_2
- no-connect marks 0 -> 2
Changed lines of the file:
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@@
 		(color 0 0 0 0)
+	)
+	(no_connect
+		(at 139.7 74.93)
+	)
+	(no_connect
+		(at 139.7 77.47)
 	)
 	(wire
@@
 		)
 	)
+	(label "V_Bus"
+		(at 153.67 105.41 0)
+		(effects
+			(font
+				(size 1.27 1.27)
+			)
+			(justify left bottom)
+		)
+	)
 	(label "CC2"
 		(at 218.44 110.49 180)
@@
 		)
 	)
-	(label "USB_DP"
-		(at 62.23 57.15 0)
-		(effects
-			(font
-				(size 1.27 1.27)
-			)
-			(justify left bottom)
-		)
-	)
 	(label "CC1"
 		(at 139.7 48.26 180)
@@
 		)
 	)
-	(label "V_Bus"
-		(at 153.67 105.41 0)
-		(effects
-			(font
-				(size 1.27 1.27)
-			)
-			(justify left bottom)
-		)
-	)
 	(label "USB_DP"
 		(at 139.7 45.72 180)
@@
 		)
 	)
-	(label "USB_DM"
-		(at 62.23 59.69 0)
-		(effects
-			(font
-				(size 1.27 1.27)
-			)
-			(justify left bottom)
-		)
-	)
 	(label "SBU2"
 		(at 140.97 123.19 180)
@@
 		)
 	)
-	(hierarchical_label "Can_H"
+	(hierarchical_label "USB_DM"
+		(shape input)
+		(at 62.23 60.96 0)
+		(effects
+			(font
+				(size 1.27 1.27)
+			)
+			(justify left)
+		)
+	)
+	(hierarchical_label "Out_1"
 		(shape input)
 		(at 166.37 115.57 0)
+		(effects
+			(font
+				(size 1.27 1.27)
+			)
+			(justify left)
+		)
+	)
+	(hierarchical_label "USB_DP"
+		(shape input)
+		(at 62.23 55.88 0)
 		(effects
 			(font
@@
 		)
 	)
-	(hierarchical_label "Can_L"
+	(hierarchical_label "Out_2"
 		(shape input)
 		(at 166.37 125.73 0)
@@
 		)
 		(instances
-			(project ""
+			(project "SensorHub_2.0"
 				(path "/9668bc71-8924-498e-982f-628f3083c8b8/a9b715b2-3c86-4c28-812a-8a4f3eb6a194"
 					(reference "U10")
@@
 		)
 		(instances
-			(project ""
+			(project "SensorHub_2.0"
 				(path "/9668bc71-8924-498e-982f-628f3083c8b8/a9b715b2-3c86-4c28-812a-8a4f3eb6a194"
 					(reference "U10")
@@
 		)
 		(instances
-			(project ""
+			(project "SensorHub_2.0"
 				(path "/9668bc71-8924-498e-982f-628f3083c8b8/a9b715b2-3c86-4c28-812a-8a4f3eb6a194"
 					(reference "U10")
@@
 		)
 		(instances
-			(project ""
+			(project "SensorHub_2.0"
 				(path "/9668bc71-8924-498e-982f-628f3083c8b8/a9b715b2-3c86-4c28-812a-8a4f3eb6a194"
 					(reference "U5")
@@
 		)
 		(instances
-			(project ""
+			(project "SensorHub_2.0"
 				(path "/9668bc71-8924-498e-982f-628f3083c8b8/a9b715b2-3c86-4c28-812a-8a4f3eb6a194"
 					(reference "U10")
@@
 		)
 		(instances
-			(project ""
+			(project "SensorHub_2.0"
 				(path "/9668bc71-8924-498e-982f-628f3083c8b8/a9b715b2-3c86-4c28-812a-8a4f3eb6a194"
 					(reference "J6")
@@
 		)
 		(instances
-			(project ""
+			(project "SensorHub_2.0"
 				(path "/9668bc71-8924-498e-982f-628f3083c8b8/a9b715b2-3c86-4c28-812a-8a4f3eb6a194"
 					(reference "U10")

Commit message: PCB 1st upd
Parts:
- added C20, C21: 0.1 uF, Capacitor_SMD:C_0603_1608Metric, symbol Device:C
Connections:
- net GND: now also C20.2, C21.2
- net V_Bus: now also C20.1, C21.1

Commit message: PCB_1.0
Connections:
- net CC1: now also U4.6 (I/O4); no longer U4.4 (I/O3)
- net CC2: now also U4.4 (I/O3); no longer U4.6 (I/O4)
- net SBU1: now also U7.3 (I/O2); no longer U7.1 (I/O1)
- net SBU2: now also U7.1 (I/O1); no longer U7.3 (I/O2)
- net USB_DM: now also U4.3 (I/O2); no longer U4.1 (I/O1)
- net USB_DP: now also U4.1 (I/O1); no longer U4.3 (I/O2)
Changed lines of the file:
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@@
 	)
 	(label "SBU1"
-		(at 139.7 69.85 180)
+		(at 139.7 72.39 180)
 		(effects
 			(font
@@
 	)
 	(label "USB_DM"
-		(at 139.7 43.18 180)
+		(at 139.7 45.72 180)
 		(effects
 			(font
@@
 	)
 	(label "SBU2"
-		(at 139.7 72.39 180)
+		(at 139.7 69.85 180)
 		(effects
 			(font
@@
 	)
 	(label "CC1"
-		(at 139.7 48.26 180)
+		(at 139.7 50.8 180)
 		(effects
 			(font
@@
 	)
 	(label "USB_DP"
-		(at 139.7 45.72 180)
+		(at 139.7 43.18 180)
 		(effects
 			(font
@@
 	)
 	(label "CC2"
-		(at 139.7 50.8 180)
+		(at 139.7 48.26 180)
 		(effects
 			(font

Commit message: Vesrion 2
Parts:
- removed U5: TMUX154EDGS, Package_SO:VSSOP-10_3x3mm_P0.5mm, symbol Analog_Switch:TMUX154EDGS
Connections:
- net cable_orient is gone; now on an unnamed net: U10.2
- net CC1: now also U4.4 (I/O3); no longer U10.5 (+), U4.6 (I/O4)
- net CC2: now also U4.6 (I/O4); no longer U10.10 (-), U4.4 (I/O3)
- net Out_1: now also J6.A8 (SBU1), J8.B8 (SBU2), U7.3 (I/O2)
- net Out_2: now also J6.B8 (SBU2), J8.A8 (SBU1), U7.1 (I/O1)
- net at R9.1, U10.1, U10.9 (+): no longer U10.13
- net at R3.1, R8.2, U10.7 (+)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: now also U10.5 (+); no longer U10.11 (+)
- removed net SBU1: J6.A8 (SBU1), J8.A8 (SBU1), U7.3 (I/O2)
- removed net SBU2: J6.B8 (SBU2), J8.B8 (SBU2), U7.1 (I/O1)
- no-connect marks 2 -> 5
Other:
- moved on the sheet: C20, C21, U10A, U10C, U10E

Commit message: MPN + CC fix
Parts:
- added R5, R6: 5.1 K, Resistor_SMD:R_0201_0603Metric, symbol Device:R
- U10: MPN (none) -> LMV339IDR
- U4, U7: MPN (none) -> USBLC6-4SC6Y
Connections:
- net CC1: now also R6.1
- net CC2: now also R5.1
- net GND: now also R5.2, R6.2

Commit message: pcb fix
Parts:
- R10, R3, R5, R6, R8, R9: footprint Resistor_SMD:R_0201_0603Metric -> Resistor_SMD:R_0402_1005Metric
Changed lines of the file:
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@@
 			)
 		)
-		(property "Footprint" "Resistor_SMD:R_0201_0603Metric"
+		(property "Footprint" "Resistor_SMD:R_0402_1005Metric"
 			(at 203.708 83.82 90)
 			(effects
@@
 			)
 		)
-		(property "Footprint" "Resistor_SMD:R_0201_0603Metric"
+		(property "Footprint" "Resistor_SMD:R_0402_1005Metric"
 			(at 80.772 133.35 90)
 			(effects
@@
 			)
 		)
-		(property "Footprint" "Resistor_SMD:R_0201_0603Metric"
+		(property "Footprint" "Resistor_SMD:R_0402_1005Metric"
 			(at 203.708 96.52 90)
 			(effects
@@
 			)
 		)
-		(property "Footprint" "Resistor_SMD:R_0201_0603Metric"
+		(property "Footprint" "Resistor_SMD:R_0402_1005Metric"
 			(at 255.778 116.84 90)
 			(effects
@@
 			)
 		)
-		(property "Footprint" "Resistor_SMD:R_0201_0603Metric"
+		(property "Footprint" "Resistor_SMD:R_0402_1005Metric"
 			(at 87.122 133.35 90)
 			(effects
@@
 			)
 		)
-		(property "Footprint" "Resistor_SMD:R_0201_0603Metric"
+		(property "Footprint" "Resistor_SMD:R_0402_1005Metric"
 			(at 235.458 86.36 90)
 			(effects

Commit message: DP/DM
Connections:
- net CC1: now also U4.6 (I/O4); no longer U4.4 (I/O3)
- net CC2: now also U7.4 (I/O3); no longer U4.6 (I/O4)
- net USB_DM: now also J8.A7 (D-), J8.B7 (D-), U4.1 (I/O1); no longer J6.A6 (D+), J6.B6 (D+), J8.A6 (D+), J8.B6 (D+), U4.3 (I/O2)
- net USB_DP: now also J8.A6 (D+), J8.B6 (D+), U4.3 (I/O2); no longer J6.A7 (D-), J6.B7 (D-), J8.A7 (D-), J8.B7 (D-), U4.1 (I/O1)
- no-connect marks 5 -> 9
