File: SensorHub/SensorHub_2.0/USB_C_2.0+SBUS.kicad_sch (KiCad schematic)
At the start: 13 parts, among them J6 USB_C_Receptacle_USB2.0_16P, J8 USB_C_Receptacle_USB2.0_16P, U10 LMV339, U4 USBLC6-4SC6, U7 USBLC6-4SC6

Commit message: v 2.3
Parts:
- removed U10: LMV339, Package_SO:SOIC-14_3.9x8.7mm_P1.27mm, symbol Comparator:LMV339
- added IC1: LM239QT, QFN50P300X300X100-17N:QFN50P300X300X100-17N, symbol LM239QT:LM239QT
- R10, R3, R5, R6, R8, R9: footprint Resistor_SMD:R_0402_1005Metric -> Resistor_SMD:R_0603_1608Metric
Connections:
- net CC1: now also U7.6 (I/O4), IC1.5 (IN-2); no longer U4.6 (I/O4)
- net CC2: now also IC1.7 (IN-3)
- net EN: now also IC1.13 (OUT4)
- net GND: now also IC1.12 (VCC-), IC1.17 (THERMALPAD), IC1.2 (IN-1), IC1.3 (NC_1), IC1.4 (IN+1)
- net USB_DM: now also J6.A7 (D-), J6.B7 (D-), U4.3 (I/O2); no longer J8.A7 (D-), J8.B7 (D-), U4.1 (I/O1)
- net USB_DP: now also J6.A6 (D+), J6.B6 (D+), U4.1 (I/O1); no longer J8.A6 (D+), J8.B6 (D+), U4.3 (I/O2)
- net V_Bus: now also IC1.1 (VCC+)
- net DIR_OUT: now reaches R9.1
- net DIR_OUT: now also IC1.11 (IN+4), IC1.14 (OUT3), IC1.15 (OUT2)
- net at R3.1, R8.2: now also IC1.6 (IN+2), IC1.8 (IN+3), IC1.9 (IN-4)
- no-connect marks 9 -> 8
Other:
- moved on the sheet: R10, R3, R8, R9, U4
