File: SensorHub/SensorHub_2.0/2.kicad_sch (KiCad schematic)
At the start: 10 parts, among them U2 MYRGM080200C41RA

Commit message: TCAN334
Changed lines of the file:
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@@
-	)
-	(label "Sleep"
-		(at 88.9 45.72 0)
-		(effects
-			(font
-				(size 1.27 1.27)
-			)
-			(justify left bottom)
-		)
 	)
 	(label "Sleep"
@@
 	(hierarchical_label "Sleep"
 		(shape input)
-		(at 76.2 80.01 0)
+		(at 88.9 45.72 0)
 		(effects
 			(font

Commit message: PCB upd 2
Connections:
- net +5V: now also D3.1 (K); no longer F1.1
- net V_Bus: now also F1.2; no longer D3.2 (A)
- new net: D3.2 (A), F1.1
Other:
- moved on the sheet: D3, F1
Changed lines of the file:
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@@
 	(symbol
 		(lib_id "Device:Fuse")
-		(at 30.48 35.56 0)
+		(at 30.48 48.26 0)
 		(unit 1)
 		(exclude_from_sim no)
@@
 		(fields_autoplaced yes)
 		(property "Reference" "F1"
-			(at 33.02 34.2899 0)
+			(at 33.02 46.9899 0)
 			(effects
 				(font
@@
 		)
 		(property "Value" "6V 0.5A"
-			(at 33.02 36.8299 0)
+			(at 33.02 49.5299 0)
 			(effects
 				(font
@@
 		)
 		(property "Footprint" "Fuse:Fuse_1206_3216Metric_Pad1.42x1.75mm_HandSolder"
-			(at 28.702 35.56 90)
+			(at 28.702 48.26 90)
 			(effects
 				(font
@@
 		)
 		(property "Datasheet" "~"
-			(at 30.48 35.56 0)
+			(at 30.48 48.26 0)
 			(effects
 				(font
@@
 		)
 		(property "Description" "Fuse"
-			(at 30.48 35.56 0)
+			(at 30.48 48.26 0)
 			(effects
 				(font
@@
 	(symbol
 		(lib_id "Diode:1N4148WT")
-		(at 30.48 48.26 270)
+		(at 30.48 35.56 270)
 		(unit 1)
 		(exclude_from_sim no)
@@
 		(fields_autoplaced yes)
 		(property "Reference" "D3"
-			(at 33.02 46.9899 90)
+			(at 33.02 34.2899 90)
 			(effects
 				(font
@@
 		)
 		(property "Value" "1N4148WT"
-			(at 33.02 49.5299 90)
+			(at 33.02 36.8299 90)
 			(effects
 				(font
@@
 		)
 		(property "Footprint" "Diode_SMD:D_SOD-523"
-			(at 26.035 48.26 0)
+			(at 26.035 35.56 0)
 			(effects
 				(font
@@
 		)
 		(property "Datasheet" "https://www.diodes.com/assets/Datasheets/ds30396.pdf"
-			(at 30.48 48.26 0)
+			(at 30.48 35.56 0)
 			(effects
 				(font
@@
 		)
 		(property "Description" "75V 0.15A Fast switching Diode, SOD-523"
-			(at 30.48 48.26 0)
+			(at 30.48 35.56 0)
 			(effects
 				(font
@@
 		)
 		(property "Sim.Device" "D"
-			(at 30.48 48.26 0)
+			(at 30.48 35.56 0)
 			(effects
 				(font
@@
 		)
 		(property "Sim.Pins" "1=K 2=A"
-			(at 30.48 48.26 0)
-			(effects
-				(font
+			(at 30.48 35.56 0)
+			(effects
+				(font

Commit message: PCB_1.0
Connections:
- net +5V: now also R1.2
- net GND: no longer R1.2
- net Sleep: no longer names the net of R1.1, U2.6 (CE)
Other:
- moved on the sheet: R1
Changed lines of the file:
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@@
 	(wire
 		(pts
-			(xy 76.2 74.93) (xy 76.2 82.55)
+			(xy 93.98 45.72) (xy 88.9 45.72)
 		)
 		(stroke
@@
 	(wire
 		(pts
-			(xy 88.9 33.02) (xy 88.9 35.56)
+			(xy 101.6 45.72) (xy 105.41 45.72)
 		)
 		(stroke
@@
 	(wire
 		(pts
-			(xy 66.04 74.93) (xy 66.04 77.47)
+			(xy 88.9 33.02) (xy 88.9 35.56)
 		)
 		(stroke
@@
 	(wire
 		(pts
-			(xy 142.24 54.61) (xy 142.24 46.99)
+			(xy 66.04 74.93) (xy 66.04 77.47)
 		)
 		(stroke
@@
 	(wire
 		(pts
-			(xy 120.65 39.37) (xy 120.65 31.75)
+			(xy 142.24 54.61) (xy 142.24 46.99)
 		)
 		(stroke
@@
 	(wire
 		(pts
-			(xy 76.2 97.79) (xy 76.2 90.17)
+			(xy 120.65 39.37) (xy 120.65 31.75)
 		)
 		(stroke
@@
 	(label "LX"
 		(at 88.9 33.02 0)
-		(effects
-			(font
-				(size 1.27 1.27)
-			)
-			(justify left bottom)
-		)
-	)
-	(label "Sleep"
-		(at 76.2 74.93 0)
 		(effects
 			(font
@@
 			)
 			(justify right)
-		)
-	)
-	(hierarchical_label "Sleep"
-		(shape input)
-		(at 88.9 45.72 0)
-		(effects
-			(font
-				(size 1.27 1.27)
-			)
-			(justify left)
 		)
 	)
@@
 	(symbol
 		(lib_id "Device:R")
-		(at 76.2 86.36 0)
+		(at 97.79 45.72 90)
 		(unit 1)
 		(exclude_from_sim no)
@@
 		(fields_autoplaced yes)
 		(property "Reference" "R1"
-			(at 78.74 85.0899 0)
-			(effects
-				(font
-					(size 1.27 1.27)
-				)
-				(justify left)
+			(at 97.79 39.37 90)
+			(effects
+				(font
+					(size 1.27 1.27)
+				)
 			)
 		)
 		(property "Value" "10 K"
-			(at 78.74 87.6299 0)
-			(effects
-				(font
-					(size 1.27 1.27)
-				)
-				(justify left)
+			(at 97.79 41.91 90)
+			(effects
+				(font
+					(size 1.27 1.27)
+				)
 			)
 		)
 		(property "Footprint" "Resistor_SMD:R_0201_0603Metric"
-			(at 74.422 86.36 90)
+			(at 97.79 47.498 90)
 			(effects
 				(font
@@
 		)
 		(property "Datasheet" "~"
-			(at 76.2 86.36 0)
+			(at 97.79 45.72 0)
 			(effects
 				(font
@@
 		)
 		(property "Description" "Resistor"
-			(at 76.2 86.36 0)
+			(at 97.79 45.72 0)
 			(effects
 				(font
@@
 	)
 	(symbol
-		(lib_id "power:GND")
-		(at 76.2 97.79 0)
-		(unit 1)
-		(exclude_from_sim no)
-		(in_bom yes)
-		(on_board yes)
-		(dnp no)
-		(fields_autoplaced yes)
-		(property "Reference" "#PWR03"
-			(at 76.2 104.14 0)
-			(effects
-				(font
-					(size 1.27 1.27)
-				)
-				(hide yes)
-			)
-		)
-		(property "Value" "GND"
-			(at 76.2 102.87 0)
-			(effects
-				(font
-					(size 1.27 1.27)
-				)
-			)
-		)
-		(property "Footprint" ""
-			(at 76.2 97.79 0)
-			(effects
-				(font
-					(size 1.27 1.27)
-				)
-				(hide yes)
-			)
-		)
-		(property "Datasheet" ""
-			(at 76.2 97.79 0)
-			(effects
-				(font
-					(size 1.27 1.27)
-				)
-				(hide yes)
-			)
-		)
-		(property "Description" "Power symbol creates a global label with name \"GND\" , ground"
-			(at 76.2 97.79 0)
-			(effects
-				(font
-					(size 1.27 1.27)
-				)
-				(hide yes)
-			)
-		)
-		(pin "1"
-		)
-		(instances
-			(project ""
-				(path "/9668bc71-8924-498e-982f-628f3083c8b8/8a6ccad9-ec56-409c-b066-b602b428230e"
-					(reference "#PWR03")
-					(unit 1)
-				)
-			)
-		)
-	)
-	(symbol
 		(lib_id "Device:C")
 		(at 142.24 43.18 0)
@@
 					(unit 1)
 				)
+			)
+		)
+	)
+	(symbol
+		(lib_id "power:+5V")
+		(at 105.41 45.72 270)
+		(unit 1)
+		(exclude_from_sim no)
+		(in_bom yes)
+		(on_board yes)
+		(dnp no)
+		(fields_autoplaced yes)
+		(property "Reference" "#PWR049"
+			(at 101.6 45.72 0)
+			(effects
+				(font
+					(size 1.27 1.27)
+				)
+				(hide yes)
+			)
+		)
+		(property "Value" "+5V"
+			(at 109.22 45.7199 90)
+			(effects
+				(font
+					(size 1.27 1.27)
+				)
+				(justify left)
+			)
+		)
+		(property "Footprint" ""
+			(at 105.41 45.72 0)
+			(effects
+				(font
+					(size 1.27 1.27)
+				)
+				(hide yes)
+			)
+		)
+		(property "Datasheet" ""
+			(at 105.41 45.72 0)
+			(effects
+				(font
+					(size 1.27 1.27)
+				)
+				(hide yes)
+			)
+		)
+		(property "Description" "Power symbol creates a global label with name \"+5V\""
+			(at 105.41 45.72 0)
+			(effects
+				(font
+					(size 1.27 1.27)
+				)
+				(hide yes)
+			)
+		)
+		(pin "1"
+		)
+		(instances
+			(project "SensorHub_2.0"
+				(path "/9668bc71-8924-498e-982f-628f3083c8b8/8a6ccad9-ec56-409c-b066-b602b428230e"
+					(reference "#PWR049")
+					(unit 1)
+				)

Commit message: JLCPCB limits
Changed lines of the file:
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@@
 					(size 1.27 1.27)
 				)
-				(hide yes)
 			)
 		)

Commit message: Vesrion 2
Parts:
- removed D3: 1N4148WT, Diode_SMD:D_SOD-523, symbol Diode:1N4148WT
Connections:
- net +5V: now also F1.1
Changed lines of the file:
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@@
-	(wire
-		(pts
-			(xy 30.48 26.67) (xy 30.48 31.75)
-		)
-		(stroke
-			(width 0)
-			(type default)
-		)
-	)
 	(wire
 		(pts
@@
 	(wire
 		(pts
-			(xy 30.48 39.37) (xy 30.48 44.45)
+			(xy 30.48 26.67) (xy 30.48 44.45)
 		)
 		(stroke
@@
 					(unit 1)
 				)
-			)
-		)
-	)
-	(symbol
-		(lib_id "Diode:1N4148WT")
-		(at 30.48 35.56 270)
-		(unit 1)
-		(exclude_from_sim no)
-		(in_bom yes)
-		(on_board yes)
-		(dnp no)
-		(fields_autoplaced yes)
-		(property "Reference" "D3"
-			(at 33.02 34.2899 90)
-			(effects
-				(font
-					(size 1.27 1.27)
-				)
-				(justify left)
-			)
-		)
-		(property "Value" "1N4148WT"
-			(at 33.02 36.8299 90)
-			(effects
-				(font
-					(size 1.27 1.27)
-				)
-				(justify left)
-			)
-		)
-		(property "Footprint" "Diode_SMD:D_SOD-523"
-			(at 26.035 35.56 0)
-			(effects
-				(font
-					(size 1.27 1.27)
-				)
-				(hide yes)
-			)
-		)
-		(property "Datasheet" "https://www.diodes.com/assets/Datasheets/ds30396.pdf"
-			(at 30.48 35.56 0)
-			(effects
-				(font
-					(size 1.27 1.27)
-				)
-				(hide yes)
-			)
-		)
-		(property "Description" "75V 0.15A Fast switching Diode, SOD-523"
-			(at 30.48 35.56 0)
-			(effects
-				(font
-					(size 1.27 1.27)
-				)
-				(hide yes)
-			)
-		)
-		(property "Sim.Device" "D"
-			(at 30.48 35.56 0)
-			(effects
-				(font
-					(size 1.27 1.27)
-				)
-				(hide yes)
-			)
-		)
-		(property "Sim.Pins" "1=K 2=A"
-			(at 30.48 35.56 0)
-			(effects
-				(font
-					(size 1.27 1.27)
-				)
-				(hide yes)
-			)
-		)
-		(pin "1"
-		)
-		(pin "2"
-		)
-		(instances
-			(project "SensorHub_2.0"
-				(path "/9668bc71-8924-498e-982f-628f3083c8b8/8a6ccad9-ec56-409c-b066-b602b428230e"
-					(reference "D3")
-					(unit 1)
-				)

Commit message: MPN + CC fix
Parts:
- F1: MPN (none) -> SMD1206B050TF
Changed lines of the file:
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@@
 			)
 		)
-		(property "Datasheet" "~"
+		(property "Datasheet" "https://nl.mouser.com/datasheet/3/508/1/SMD1206_1.pdf"
 			(at 30.48 48.26 0)
 			(effects
@@
 			)
 		)
+		(property "MPN" "SMD1206B050TF "
+			(at 30.48 48.26 0)
+			(effects
+				(font
+					(size 1.27 1.27)
+				)
+				(hide yes)
+			)
+		)
 		(pin "1"
 		)
@@
 			)
 		)
-		(property "Datasheet" ""
+		(property "Datasheet" "https://nl.mouser.com/datasheet/3/76/2/MYRGM_c_x.pdf"
 			(at 58.42 25.4 0)
 			(effects

Commit message: pcb fix
Parts:
- R1, R12, R2: footprint Resistor_SMD:R_0201_0603Metric -> Resistor_SMD:R_0402_1005Metric
Changed lines of the file:
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@@
 			)
 		)
-		(property "Footprint" "Resistor_SMD:R_0201_0603Metric"
+		(property "Footprint" "Resistor_SMD:R_0402_1005Metric"
 			(at 64.262 81.28 90)
 			(effects
@@
 			)
 		)
-		(property "Footprint" "Resistor_SMD:R_0201_0603Metric"
+		(property "Footprint" "Resistor_SMD:R_0402_1005Metric"
 			(at 64.262 91.44 90)
 			(effects
@@
 			)
 		)
-		(property "Footprint" "Resistor_SMD:R_0201_0603Metric"
+		(property "Footprint" "Resistor_SMD:R_0402_1005Metric"
 			(at 97.79 47.498 90)
 			(effects

Commit message: v 2.3
Parts:
- R1, R12, R2: footprint Resistor_SMD:R_0402_1005Metric -> Resistor_SMD:R_0603_1608Metric
- U2: footprint MYRGM080200C41RA:MURATA_MYRGM080200C41RA_0 -> MURATA_MYRGM080200C41RA_0:MURATA_MYRGM080200C41RA_0
Changed lines of the file:
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@@
 			)
 		)
-		(property "Footprint" "Resistor_SMD:R_0402_1005Metric"
+		(property "Footprint" "Resistor_SMD:R_0603_1608Metric"
 			(at 64.262 81.28 90)
 			(effects
@@
 			)
 		)
-		(property "Footprint" "Resistor_SMD:R_0402_1005Metric"
+		(property "Footprint" "Resistor_SMD:R_0603_1608Metric"
 			(at 64.262 91.44 90)
 			(effects
@@
 			)
 		)
-		(property "Footprint" "Resistor_SMD:R_0402_1005Metric"
+		(property "Footprint" "Resistor_SMD:R_0603_1608Metric"
 			(at 97.79 47.498 90)
 			(effects
@@
 			)
 		)
-		(property "Footprint" "MYRGM080200C41RA:MURATA_MYRGM080200C41RA_0"
+		(property "Footprint" "MURATA_MYRGM080200C41RA_0:MURATA_MYRGM080200C41RA_0"
 			(at 58.42 25.4 0)
 			(effects
