File: SensorHub/SensorHub_2.0/LSM6DSM_IMU.kicad_sch (KiCad schematic)
At the start: 3 parts, among them U6 LSM6DSM

Commit message: PCB_1.0
Parts:
- removed TP9: TestPoint, TestPoint:TestPoint_THTPad_D1.0mm_Drill0.5mm, symbol Connector:TestPoint
Changed lines of the file:
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@@
-		(color 0 0 0 0)
-	)
-	(junction
-		(at 88.9 100.33)
-		(diameter 0)
 		(color 0 0 0 0)
 	)
@@
 	(wire
 		(pts
-			(xy 88.9 100.33) (xy 92.71 100.33)
+			(xy 87.63 100.33) (xy 92.71 100.33)
 		)
 		(stroke
@@
 		(pts
 			(xy 92.71 90.17) (xy 92.71 92.71)
-		)
-		(stroke
-			(width 0)
-			(type default)
-		)
-	)
-	(wire
-		(pts
-			(xy 87.63 100.33) (xy 88.9 100.33)
 		)
 		(stroke
@@
 					(unit 1)
 				)
-			)
-		)
-	)
-	(symbol
-		(lib_id "Connector:TestPoint")
-		(at 88.9 100.33 180)
-		(unit 1)
-		(exclude_from_sim no)
-		(in_bom yes)
-		(on_board yes)
-		(dnp no)
-		(property "Reference" "TP9"
-			(at 93.472 108.712 0)
-			(effects
-				(font
-					(size 1.27 1.27)
-				)
-				(justify left)
-			)
-		)
-		(property "Value" "TestPoint"
-			(at 93.472 107.1881 0)
-			(effects
-				(font
-					(size 1.27 1.27)
-				)
-				(justify left)
-				(hide yes)
-			)
-		)
-		(property "Footprint" "TestPoint:TestPoint_THTPad_D1.0mm_Drill0.5mm"
-			(at 83.82 100.33 0)
-			(effects
-				(font
-					(size 1.27 1.27)
-				)
-				(hide yes)
-			)
-		)
-		(property "Datasheet" "~"
-			(at 83.82 100.33 0)
-			(effects
-				(font
-					(size 1.27 1.27)
-				)
-				(hide yes)
-			)
-		)
-		(property "Description" "test point"
-			(at 88.9 100.33 0)
-			(effects
-				(font
-					(size 1.27 1.27)
-				)
-				(hide yes)
-			)
-		)
-		(pin "1"
-		)
-		(instances
-			(project "SensorHub_2.0"
-				(path "/9668bc71-8924-498e-982f-628f3083c8b8/cfff8b62-f604-412e-84a3-6cd10c96a62b"
-					(reference "TP9")
-					(unit 1)
-				)

Commit message: MPN + CC fix
Parts:
- U6: MPN (none) -> LSM6DSMTR
Changed lines of the file:
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@@
 			)
 		)
-		(property "Datasheet" ""
+		(property "Datasheet" "https://www.st.com/resource/en/datasheet/lsm6dsm.pdf"
 			(at 115.57 90.17 0)
 			(effects
@@
 				(hide yes)
 			)
+		)
+		(property "MPN" "LSM6DSMTR"
+			(at 115.57 90.17 0)
+			(effects
+				(font
+					(size 1.27 1.27)
+				)
+				(hide yes)
+			)

Commit message: v 2.3
Parts:
- U6: footprint LSM6DSM:PQFN50P300X250X86-14N -> PQFN50P300X250X86-14N:PQFN50P300X250X86-14N
Changed lines of the file:
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@@
 			)
 		)
-		(property "Footprint" "LSM6DSM:PQFN50P300X250X86-14N"
+		(property "Footprint" "PQFN50P300X250X86-14N:PQFN50P300X250X86-14N"
 			(at 115.57 90.17 0)
 			(effects
