File: Compressions/CompressionSensor_2.0/CompressionSensor_2.0.kicad_sch (KiCad schematic)
At the start: 12 parts, among them J5 658511223020, U1 VL53L4CD

Commit message: Sensors
Parts:
- removed D1: RED, Compressions_TOF_VL53L4CD_v1.0.0_mar2025:LED-0603, symbol Compressions_TOF_VL53L4CD_v1.0.0_mar2025-eagle-import:LED-RED0603
- added D2: LED, LED_SMD:LED_0603_1608Metric, symbol Device:LED
- C1, C4: footprint Compressions_TOF_VL53L4CD_v1.0.0_mar2025:0603 -> Capacitor_SMD:C_0603_1608Metric
- C2, C3: footprint Compressions_TOF_VL53L4CD_v1.0.0_mar2025:0805-NO -> Capacitor_SMD:C_0603_1608Metric
- R1, R2, R3: footprint Compressions_TOF_VL53L4CD_v1.0.0_mar2025:0603 -> Resistor_SMD:R_0603_1608Metric
Connections:
- net +3.3V is gone; now on net 3.3V: J5.19
- net GP1 is gone; now on net ~{SHUT}: J5.14
- net INT2 is gone; now on net ~{INT}: J5.15
- net SCL_0 is gone; now on net SCL: J5.9
- net SDA_0 is gone; now on net SDA: J5.7
- net at R3.1: now also D2.2 (A)
- net at PWR0.2: now also D2.1 (K)
- net +5V: no longer names the net of J5.12
- no-connect marks 4 -> 6
